File: AlarmClock/ambient.sch (KiCad schematic (older format))
At the start: 12 parts

Commit message: Annotate schematics, assign footprints, pcbnew
Parts:
- C12: renamed from C?; value 100u -> 100u / 16V; footprint (none) -> Capacitor_SMD:CP_Elec_6.3x5.4; GES (none) -> GES05413805
- C13: renamed from C?; footprint (none) -> Capacitor_SMD:C_1206_3216Metric_Pad1.33x1.80mm_HandSolder
- D6: renamed from D?; footprint (none) -> Connector_Molex:Molex_KK-254_AE-6410-02A_1x02_P2.54mm_Vertical
- R17, R18, R19, R20, R21: renamed from R?; footprint (none) -> Resistor_SMD:R_1206_3216Metric_Pad1.30x1.75mm_HandSolder
- gave numbers to parts that had none: 4
Changed lines of the file:
@@
 ambient
 $Comp
-L Device:R R?
+L Device:R R17
 U 1 1 621AB628
 P 4750 3500
-F 0 "R?" V 4543 3500 50  0000 C CNN
+F 0 "R17" V 4543 3500 50  0000 C CNN
 F 1 "1k" V 4634 3500 50  0000 C CNN
-F 2 "" V 4680 3500 50  0001 C CNN
+F 2 "Resistor_SMD:R_1206_3216Metric_Pad1.30x1.75mm_HandSolder" V 4680 3500 50  0001 C CNN
 F 3 "~" H 4750 3500 50  0001 C CNN
 	1    4750 3500
@@
 $EndComp
 $Comp
-L Device:R R?
+L Device:R R18
 U 1 1 621AC01B
 P 5250 3500
-F 0 "R?" V 5043 3500 50  0000 C CNN
+F 0 "R18" V 5043 3500 50  0000 C CNN
 F 1 "10k" V 5134 3500 50  0000 C CNN
-F 2 "" V 5180 3500 50  0001 C CNN
+F 2 "Resistor_SMD:R_1206_3216Metric_Pad1.30x1.75mm_HandSolder" V 5180 3500 50  0001 C CNN
 F 3 "~" H 5250 3500 50  0001 C CNN
 	1    5250 3500
@@
 $EndComp
 $Comp
-L Device:CP C?
+L Device:CP C12
 U 1 1 621AC648
 P 5000 3750
-F 0 "C?" H 5118 3796 50  0000 L CNN
-F 1 "100u" H 5118 3705 50  0000 L CNN
-F 2 "" H 5038 3600 50  0001 C CNN
+F 0 "C12" H 4750 3750 50  0000 L CNN
+F 1 "100u / 16V" H 4500 3650 50  0000 L CNN
+F 2 "Capacitor_SMD:CP_Elec_6.3x5.4" H 5038 3600 50  0001 C CNN
 F 3 "~" H 5000 3750 50  0001 C CNN
+F 4 "GES05413805" H 5000 3750 50  0001 C CNN "GES"
 	1    5000 3750
 	1    0    0    -1
@@
 $EndComp
 $Comp
-L Device:R R?
+L Device:R R20
 U 1 1 621AD2C2
 P 5500 3750
-F 0 "R?" H 5570 3796 50  0000 L CNN
+F 0 "R20" H 5570 3796 50  0000 L CNN
 F 1 "10k" H 5570 3705 50  0000 L CNN
-F 2 "" V 5430 3750 50  0001 C CNN
+F 2 "Resistor_SMD:R_1206_3216Metric_Pad1.30x1.75mm_HandSolder" V 5430 3750 50  0001 C CNN
 F 3 "~" H 5500 3750 50  0001 C CNN
 	1    5500 3750
@@
 $EndComp
 $Comp
-L Device:R R?
+L Device:R R19
 U 1 1 621AD605
 P 5500 3250
-F 0 "R?" H 5570 3296 50  0000 L CNN
+F 0 "R19" H 5570 3296 50  0000 L CNN
 F 1 "22k" H 5570 3205 50  0000 L CNN
-F 2 "" V 5430 3250 50  0001 C CNN
+F 2 "Resistor_SMD:R_1206_3216Metric_Pad1.30x1.75mm_HandSolder" V 5430 3250 50  0001 C CNN
 F 3 "~" H 5500 3250 50  0001 C CNN
 	1    5500 3250
@@
 $EndComp
 $Comp
-L Transistor_BJT:BCP56 Q?
+L Transistor_BJT:BCP56 Q8
 U 1 1 621B0128
 P 7400 3500
-F 0 "Q?" H 7591 3546 50  0000 L CNN
+F 0 "Q8" H 7591 3546 50  0000 L CNN
 F 1 "BCP56" H 7591 3455 50  0000 L CNN
 F 2 "Package_TO_SOT_SMD:SOT-223-3_TabPin2" H 7600 3425 50  0001 L CIN
@@
 $EndComp
 $Comp
-L Transistor_BJT:BC847 Q?
+L Transistor_BJT:BC847 Q7
 U 1 1 621B1718
 P 6900 3250
-F 0 "Q?" H 7091 3296 50  0000 L CNN
+F 0 "Q7" H 7091 3296 50  0000 L CNN
 F 1 "BC847" H 7091 3205 50  0000 L CNN
 F 2 "Package_TO_SOT_SMD:SOT-23" H 7100 3175 50  0001 L CIN
@@
 $EndComp
 $Comp
-L Transistor_BJT:BC847 Q?
+L Transistor_BJT:BC847 Q6
 U 1 1 621B2E67
 P 6600 3750
-F 0 "Q?" H 6791 3796 50  0000 L CNN
+F 0 "Q6" H 6791 3796 50  0000 L CNN
 F 1 "BC847" H 6791 3705 50  0000 L CNN
 F 2 "Package_TO_SOT_SMD:SOT-23" H 6800 3675 50  0001 L CIN
@@
 Connection ~ 5500 3500
 $Comp
-L Device:R R?
+L Device:R R21
 U 1 1 621B6EB3
 P 7500 4250
-F 0 "R?" H 7570 4296 50  0000 L CNN
+F 0 "R21" H 7570 4296 50  0000 L CNN
 F 1 "6R8" H 7570 4205 50  0000 L CNN
-F 2 "" V 7430 4250 50  0001 C CNN
+F 2 "Resistor_SMD:R_1206_3216Metric_Pad1.30x1.75mm_HandSolder" V 7430 4250 50  0001 C CNN
 F 3 "~" H 7500 4250 50  0001 C CNN
 	1    7500 4250
@@
 	7500 3000 7500 3300
 $Comp
-L Device:LED D?
+L Device:LED D6
 U 1 1 621B87DD
 P 7500 2750
-F 0 "D?" V 7539 2632 50  0000 R CNN
+F 0 "D6" V 7539 2632 50  0000 R CNN
 F 1 "LED" V 7448 2632 50  0000 R CNN
-F 2 "" H 7500 2750 50  0001 C CNN
+F 2 "Connector_Molex:Molex_KK-254_AE-6410-02A_1x02_P2.54mm_Vertical" H 7500 2750 50  0001 C CNN
 F 3 "~" H 7500 2750 50  0001 C CNN
 	1    7500 2750
@@
 	5500 3500 5850 3500
 $Comp
-L Diode:1N4148W D?
+L Diode:1N4148W D5
 U 1 1 621BA45B
 P 6500 4250
-F 0 "D?" V 6546 4170 50  0000 R CNN
+F 0 "D5" V 6546 4170 50  0000 R CNN
 F 1 "1N4148W" V 6455 4170 50  0000 R CNN
 F 2 "Diode_SMD:D_SOD-123" H 6500 4075 50  0001 C CNN
@@
 	5500 3000 5500 3100
 $Comp
-L Device:C C?
+L Device:C C13
 U 1 1 621E5909
 P 5850 3750
-F 0 "C?" H 5965 3796 50  0000 L CNN
+F 0 "C13" H 5965 3796 50  0000 L CNN
 F 1 "100n" H 5965 3705 50  0000 L CNN
-F 2 "" H 5888 3600 50  0001 C CNN
+F 2 "Capacitor_SMD:C_1206_3216Metric_Pad1.33x1.80mm_HandSolder" H 5888 3600 50  0001 C CNN
 F 3 "~" H 5850 3750 50  0001 C CNN
 	1    5850 3750

Commit message: Fix ambient LED staying lit
Parts:
- added R27: 10k, Resistor_SMD:R_1206_3216Metric_Pad1.30x1.75mm_HandSolder, symbol Device:R
Connections:
- net +5V: now also R27.1
- net at D6.1 (K), Q7.3 (C), Q8.2 (C)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: now also R27.2
Other:
- note added: "Notes:\n- R27 is needed for the LED to fully turn off."
Changed lines of the file:
@@
 Connection ~ 7500 3000
 Wire Wire Line
-	7500 2600 7500 2500
+	7500 2600 7500 2550
 Wire Wire Line
 	6500 3550 6500 3500
@@
 Wire Wire Line
 	5850 3500 6500 3500
+$Comp
+L Device:R R27
+U 1 1 6246D589
+P 8000 2750
+F 0 "R27" H 8070 2796 50  0000 L CNN
+F 1 "10k" H 8070 2705 50  0000 L CNN
+F 2 "Resistor_SMD:R_1206_3216Metric_Pad1.30x1.75mm_HandSolder" V 7930 2750 50  0001 C CNN
+F 3 "~" H 8000 2750 50  0001 C CNN
+	1    8000 2750
+	1    0    0    -1
+$EndComp
+Wire Wire Line
+	8000 2900 8000 3000
+Wire Wire Line
+	8000 3000 7500 3000
+Wire Wire Line
+	8000 2600 8000 2550
+Wire Wire Line
+	8000 2550 7500 2550
+Connection ~ 7500 2550
+Wire Wire Line
+	7500 2550 7500 2500
+Text Notes 500  7750 0    50   ~ 0
+Notes:\n- R27 is needed for the LED to fully turn off.
 $EndSCHEMATC

Commit message: Update symbol fields for BOM
Parts:
- C13: GES (none) -> GES05400125
- Q8: TME (none) -> https://www.tme.eu/cz/details/bcp56-16tx/tranzistory-npn-sm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; TME Symbol (none) -> BCP56-16TX
- R21: TME (none) -> https://www.tme.eu/cz/details/smd1206-6r8-1%25/rezistory-sm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; TME Symbol (none) -> SMD1206-6R8-1%
Changed lines of the file:
@@
 F 2 "Package_TO_SOT_SMD:SOT-223-3_TabPin2" H 7600 3425 50  0001 L CIN
 F 3 "http://cache.nxp.com/documents/data_sheet/BCP56_BCX56_BC56PA.pdf?pspll=1" H 7400 3500 50  0001 L CNN
+F 4 "https://www.tme.eu/cz/details/bcp56-16tx/tranzistory-npn-smd/nexperia/" H 7400 3500 50  0001 C CNN "TME"
+F 5 "BCP56-16TX" H 7400 3500 50  0001 C CNN "TME Symbol"
 	1    7400 3500
 	1    0    0    -1
@@
 F 2 "Resistor_SMD:R_1206_3216Metric_Pad1.30x1.75mm_HandSolder" V 7430 4250 50  0001 C CNN
 F 3 "~" H 7500 4250 50  0001 C CNN
+F 4 "https://www.tme.eu/cz/details/smd1206-6r8-1%25/rezistory-smd-1206/royal-ohm/1206s4f680kt5e/" H 7500 4250 50  0001 C CNN "TME"
+F 5 "SMD1206-6R8-1%" H 7500 4250 50  0001 C CNN "TME Symbol"
 	1    7500 4250
 	1    0    0    -1
@@
 F 2 "Capacitor_SMD:C_1206_3216Metric_Pad1.33x1.80mm_HandSolder" H 5888 3600 50  0001 C CNN
 F 3 "~" H 5850 3750 50  0001 C CNN
+F 4 "GES05400125" H 5850 3750 50  0001 C CNN "GES"
 	1    5850 3750
 	1    0    0    -1
